File: RainMaker.kicad_pcb (KiCad board)
At the start: 2 copper layers, 130 x 72 mm, 78 parts, among them IC1 ESP32-WROOM-32D, J1 Screw Terminal - 2P, Q1 IRLR8726TRPBF, Q10 IRLR8726TRPBF, Q11 IRLR8726TRPBF, Q12 IRLR8726TRPBF, Q2 IRLR8726TRPBF, Q3 IRLR8726TRPBF, Q4 IRLR8726TRPBF, Q5 IRLR8726TRPBF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

Commit message: fix unconnected
Routing:
- net /Z_5_OUT: track 14.4 -> 18.5 mm
Changed lines of the file:
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@@
   (segment (start 87.485 102.665) (end 87.485 109.035) (width 1.5) (layer "F.Cu") (net 8))
   (segment (start 87.485 109.035) (end 94.6 116.15) (width 1.5) (layer "F.Cu") (net 8))
+  (segment (start 97.285 102.665) (end 97.285 99.668676) (width 1.5) (layer "F.Cu") (net 9))
+  (segment (start 97.285 99.668676) (end 98.053676 98.9) (width 1.5) (layer "F.Cu") (net 9))
   (segment (start 97.285 102.665) (end 97.285 113.835) (width 1.5) (layer "F.Cu") (net 9))
   (segment (start 97.285 113.835) (end 99.6 116.15) (width 1.5) (layer "F.Cu") (net 9))

Commit message: fixes
Parts:
- J3: renamed from ZONE OUT CONNECTOR1
- renumbered PROG1 to J2, IC1 to U2
Other:
- board text added: "+24V"
- board text added: "."
- board text added: "3.3V"
- board text added: "EN"
- board text added: "IO_0"
- board text added: "J2"
- board text added: "J3"
- board text added: "RX"
- board text added: "TX"
- board text added: "V1.0 01-01-2024"

Commit message: production files
Routing:
- net GND: vias 0 -> 5
Changed lines of the file:
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@@
   )
   (setup
+    (stackup
+      (layer "F.SilkS" (type "Top Silk Screen"))
+      (layer "F.Paste" (type "Top Solder Paste"))
+      (layer "F.Mask" (type "Top Solder Mask") (thickness 0.01))
+      (layer "F.Cu" (type "copper") (thickness 0.035))
+      (layer "dielectric 1" (type "core") (thickness 1.51) (material "FR4") (epsilon_r 4.5) (loss_tangent 0.02))
+      (layer "B.Cu" (type "copper") (thickness 0.035))
+      (layer "B.Mask" (type "Bottom Solder Mask") (thickness 0.01))
+      (layer "B.Paste" (type "Bottom Solder Paste"))
+      (layer "B.SilkS" (type "Bottom Silk Screen"))
+      (copper_finish "None")
+      (dielectric_constraints no)
+    )
     (pad_to_mask_clearance 0)
     (pcbplotparams
@@
     (property "ki_keywords" "capacitor cap")
     (attr smd)
-    (fp_text reference "C10" (at 3.1625 0.025) (layer "F.SilkS")
+    (fp_text reference "C10" (at 8.3875 -2.85) (layer "F.SilkS")
         (effects (font (size 1 1) (thickness 0.15)))
     )
@@
     (pad "39" smd rect (at -2.205 -2.435) (size 1.05 1.05) (layers "F.Cu" "F.Paste")
       (net 2 "GND") (pinfunction "GND") (pintype "passive"))
-    (pad "39" thru_hole circle (at -2.205 -1.6725) (size 0.6 0.6) (drill 0.2) (property pad_prop_heatsink) (layers "*.Cu" "F.Mask")
-      (net 2 "GND") (pinfunction "GND") (pintype "passive"))
     (pad "39" smd rect (at -2.205 -0.91) (size 1.05 1.05) (layers "F.Cu" "F.Paste")
       (net 2 "GND") (pinfunction "GND") (pintype "passive"))
-    (pad "39" thru_hole circle (at -2.205 -0.1475) (size 0.6 0.6) (drill 0.2) (property pad_prop_heatsink) (layers "*.Cu" "F.Mask")
-      (net 2 "GND") (pinfunction "GND") (pintype "passive"))
     (pad "39" smd rect (at -2.205 0.615) (size 1.05 1.05) (layers "F.Cu" "F.Paste")
       (net 2 "GND") (pinfunction "GND") (pintype "passive"))
-    (pad "39" thru_hole circle (at -1.4425 -2.435) (size 0.6 0.6) (drill 0.2) (property pad_prop_heatsink) (layers "*.Cu" "F.Mask")
-      (net 2 "GND") (pinfunction "GND") (pintype "passive"))
-    (pad "39" thru_hole circle (at -1.4425 -0.91) (size 0.6 0.6) (drill 0.2) (property pad_prop_heatsink) (layers "*.Cu" "F.Mask")
-      (net 2 "GND") (pinfunction "GND") (pintype "passive"))
-    (pad "39" thru_hole circle (at -1.4425 0.615) (size 0.6 0.6) (drill 0.2) (property pad_prop_heatsink) (layers "*.Cu" "F.Mask")
-      (net 2 "GND") (pinfunction "GND") (pintype "passive"))
     (pad "39" smd rect (at -0.68 -2.435) (size 1.05 1.05) (layers "F.Cu" "F.Paste")
       (net 2 "GND") (pinfunction "GND") (pintype "passive"))
-    (pad "39" thru_hole circle (at -0.68 -1.6725) (size 0.6 0.6) (drill 0.2) (property pad_prop_heatsink) (layers "*.Cu" "F.Mask")
-      (net 2 "GND") (pinfunction "GND") (pintype "passive"))
     (pad "39" smd rect (at -0.68 -0.91) (size 1.05 1.05) (layers "F.Cu" "F.Paste")
       (net 2 "GND") (pinfunction "GND") (pintype "passive"))
     (pad "39" smd rect (at -0.68 -0.91) (size 4.2 4.2) (layers "F.Cu" "F.Mask")
       (net 2 "GND") (pinfunction "GND") (pintype "passive"))
-    (pad "39" thru_hole circle (at -0.68 -0.1475) (size 0.6 0.6) (drill 0.2) (property pad_prop_heatsink) (layers "*.Cu" "F.Mask")
-      (net 2 "GND") (pinfunction "GND") (pintype "passive"))
     (pad "39" smd rect (at -0.68 0.615) (size 1.05 1.05) (layers "F.Cu" "F.Paste")
       (net 2 "GND") (pinfunction "GND") (pintype "passive"))
-    (pad "39" thru_hole circle (at 0.0825 -2.435) (size 0.6 0.6) (drill 0.2) (property pad_prop_heatsink) (layers "*.Cu" "F.Mask")
-      (net 2 "GND") (pinfunction "GND") (pintype "passive"))
-    (pad "39" thru_hole circle (at 0.0825 -0.91) (size 0.6 0.6) (drill 0.2) (property pad_prop_heatsink) (layers "*.Cu" "F.Mask")
-      (net 2 "GND") (pinfunction "GND") (pintype "passive"))
-    (pad "39" thru_hole circle (at 0.0825 0.615) (size 0.6 0.6) (drill 0.2) (property pad_prop_heatsink) (layers "*.Cu" "F.Mask")
-      (net 2 "GND") (pinfunction "GND") (pintype "passive"))
     (pad "39" smd rect (at 0.845 -2.435) (size 1.05 1.05) (layers "F.Cu" "F.Paste")
       (net 2 "GND") (pinfunction "GND") (pintype "passive"))
-    (pad "39" thru_hole circle (at 0.845 -1.6725) (size 0.6 0.6) (drill 0.2) (property pad_prop_heatsink) (layers "*.Cu" "F.Mask")
-      (net 2 "GND") (pinfunction "GND") (pintype "passive"))
     (pad "39" smd rect (at 0.845 -0.91) (size 1.05 1.05) (layers "F.Cu" "F.Paste")
       (net 2 "GND") (pinfunction "GND") (pintype "passive"))
-    (pad "39" thru_hole circle (at 0.845 -0.1475) (size 0.6 0.6) (drill 0.2) (property pad_prop_heatsink) (layers "*.Cu" "F.Mask")
-      (net 2 "GND") (pinfunction "GND") (pintype "passive"))
     (pad "39" smd rect (at 0.845 0.615) (size 1.05 1.05) (layers "F.Cu" "F.Paste")
       (net 2 "GND") (pinfunction "GND") (pintype "passive"))
@@
     )
   )
+  (gr_line (start 74.55 55.8) (end 75.05 55.325)
+    (stroke (width 0.15) (type default)) (layer "F.SilkS"))
+  (gr_line (start 79.475 54.4) (end 82.025 54.4)
+    (stroke (width 0.15) (type default)) (layer "F.SilkS"))
+  (gr_line (start 74.55 55.8) (end 75.125 55.975)
+    (stroke (width 0.15) (type default)) (layer "F.SilkS"))
+  (gr_line (start 79.475 54.4) (end 74.55 55.8)
+    (stroke (width 0.15) (type default)) (layer "F.SilkS"))
+  (gr_line (start 75.05 55.325) (end 74.55 55.8)
+    (stroke (width 0.15) (type default)) (layer "F.SilkS"))
+  (gr_line (start 82.025 54.4) (end 79.475 54.4)
+    (stroke (width 0.15) (type default)) (layer "F.SilkS"))
   (gr_arc (start 180 117) (mid 178.535534 120.535534) (end 175 122)
     (stroke (width 0.1) (type default)) (layer "Edge.Cuts"))
@@
   (segment (start 67.872476 88.125) (end 67.872476 90.90992) (width 1) (layer "F.Cu") (net 2))
   (segment (start 67.872476 90.90992) (end 67.857396 90.925) (width 1) (layer "F.Cu") (net 2))
+  (via (at 134.575 63.925) (size 0.8) (drill 0.4) (layers "F.Cu" "B.Cu") (net 2))
+  (via (at 132.325 66.15) (size 0.8) (drill 0.4) (layers "F.Cu" "B.Cu") (net 2))
+  (via (at 132.375 63.9) (size 0.8) (drill 0.4) (layers "F.Cu" "B.Cu") (net 2))
+  (via (at 133.45 65.075) (size 0.8) (drill 0.4) (layers "F.Cu" "B.Cu") (net 2))
+  (via (at 134.55 66.125) (size 0.8) (drill 0.4) (layers "F.Cu" "B.Cu") (net 2))
   (segment (start 111.415 102.665) (end 112.785 102.665) (width 2) (layer "F.Cu") (net 3))
   (segment (start 152.485 102.665) (end 152.5 102.65) (width 2) (layer "F.Cu") (net 3))
@@
   (segment (start 165.972476 86.475) (end 170.572476 86.475) (width 1) (layer "F.Cu") (net 45))
   (segment (start 147.277476 67.78) (end 165.972476 86.475) (width 0.3) (layer "F.Cu") (net 45))
-  (segment (start 145.75 64.9) (end 145.8 64.95) (width 0.3) (layer "F.Cu") (net 47))
-  (segment (start 145.8 64.95) (end 152.025 64.95) (width 0.3) (layer "F.Cu") (net 47))
+  (segment (start 144 63.97) (end 144.98 64.95) (width 0.3) (layer "F.Cu") (net 47))
   (segment (start 142.95 63.97) (end 144 63.97) (width 0.3) (layer "F.Cu") (net 47))
-  (segment (start 144 63.97) (end 144.93 64.9) (width 0.3) (layer "F.Cu") (net 47))
-  (segment (start 144.93 64.9) (end 145.75 64.9) (width 0.3) (layer "F.Cu") (net 47))
+  (segment (start 144.98 64.95) (end 152.025 64.95) (width 0.3) (layer "F.Cu") (net 47))
   (segment (start 148.835 60.16) (end 152.025 63.35) (width 0.3) (layer "F.Cu") (net 48))
   (segment (start 142.95 60.16) (end 148.835 60.16) (width 0.3) (layer "F.Cu") (net 48))
