File: RainMaker.kicad_sch (KiCad schematic)
At the start: 74 parts, among them IC1 ESP32-WROOM-32D, J1 Screw Terminal - 2P, Q1 IRLR8726TRPBF, Q10 IRLR8726TRPBF, Q11 IRLR8726TRPBF, Q12 IRLR8726TRPBF, Q2 IRLR8726TRPBF, Q3 IRLR8726TRPBF, Q4 IRLR8726TRPBF, Q5 IRLR8726TRPBF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

Commit message: fix vcc
Changed lines of the file:
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@@
     (stroke (width 0) (type default))
   )
-  (wire (pts (xy 58.42 25.4) (xy 58.42 33.02))
+  (wire (pts (xy 58.42 27.94) (xy 58.42 33.02))
     (stroke (width 0) (type default))
   )
@@
     (stroke (width 0) (type default))
   )
-  (wire (pts (xy 58.42 25.4) (xy 81.28 25.4))
+  (wire (pts (xy 58.42 27.94) (xy 81.28 27.94))
     (stroke (width 0) (type default))
   )
@@
     (effects (font (size 1.27 1.27)) (justify left bottom))
   )
-  (label "Z_1_OUT" (at 58.42 25.4 0) (fields_autoplaced)
-    (effects (font (size 1.27 1.27)) (justify left bottom))
-  )
+  (label "Z_1_OUT" (at 58.42 27.94 0) (fields_autoplaced)
+    (effects (font (size 1.27 1.27)) (justify left bottom))
+  )

Commit message: fixes
Parts:
- J3: renamed from ZONE OUT CONNECTOR1
- renumbered PROG1 to J2, IC1 to U2
Changed lines of the file:
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@@
   (symbol (lib_id "Connector_Generic:Conn_01x06") (at 353.06 92.71 0) (unit 1)
     (in_bom yes) (on_board yes) (dnp no) (fields_autoplaced)
-    (property "Reference" "PROG1" (at 355.6 92.71 0)
+    (property "Reference" "J2" (at 355.6 92.71 0)
       (effects (font (size 1.27 1.27)) (justify left))
     )
@@
       (project "RainMaker"
         (path "/524c1494-4c03-4fd8-9133-1e33af151a83"
-          (reference "PROG1") (unit 1)
+          (reference "J2") (unit 1)
         )
       )
@@
   (symbol (lib_id "easyeda2kicad:DB128V-5.0-15P") (at 353.06 151.13 0) (unit 1)
     (in_bom yes) (on_board yes) (dnp no)
-    (property "Reference" "ZONE OUT CONNECTOR1" (at 355.6 147.32 0)
+    (property "Reference" "J3" (at 355.6 147.32 0)
       (effects (font (size 1.27 1.27)) (justify left))
     )
@@
       (project "RainMaker"
         (path "/524c1494-4c03-4fd8-9133-1e33af151a83"
-          (reference "ZONE OUT CONNECTOR1") (unit 1)
+          (reference "J3") (unit 1)
         )
       )
@@
   (symbol (lib_id "RF_Module:ESP32-WROOM-32") (at 224.79 138.43 0) (unit 1)
     (in_bom yes) (on_board yes) (dnp no)
-    (property "Reference" "IC1" (at 218.44 104.14 0)
+    (property "Reference" "U2" (at 218.44 104.14 0)
       (effects (font (size 1.27 1.27)) (justify left))
     )
@@
       (project "RainMaker"
         (path "/524c1494-4c03-4fd8-9133-1e33af151a83"
-          (reference "IC1") (unit 1)
-        )
-      )
+          (reference "U2") (unit 1)
+        )
+      )

Commit message: production files
Parts:
- C10, C8, C9: LCSC (none) -> C45783
Changed lines of the file:
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@@
+      (effects (font (size 1.27 1.27)) hide)
+    )
+    (property "LCSC" "C45783" (at 261.62 46.99 0)
       (effects (font (size 1.27 1.27)) hide)
     )
@@
       (effects (font (size 1.27 1.27)) hide)
     )
+    (property "LCSC" "C45783" (at 269.24 46.99 0)
+      (effects (font (size 1.27 1.27)) hide)
+    )
     (pin "2")
     (pin "1")
@@
       (effects (font (size 1.27 1.27)) hide)
     )
-    (property "Datasheet" "~" (at 254 46.99 0)
+    (property "Datasheet" "https://www.lcsc.com/product-detail/Multilayer-Ceramic-Capacitors-MLCC-SMD-SMT_Samsung-Electro-Mechanics-CL21A226MAQNNNE_C45783.html" (at 254 46.99 0)
+      (effects (font (size 1.27 1.27)) hide)
+    )
+    (property "LCSC" "C45783" (at 254 46.99 0)
       (effects (font (size 1.27 1.27)) hide)
     )
@@
       (effects (font (size 1.27 1.27)) hide)
     )
-    (property "Datasheet" "" (at 242.57 43.18 0)
-      (effects (font (size 1.27 1.27)) hide)
-    )
+    (property "Datasheet" "https://www.lcsc.com/product-detail/Inductors-SMD_SHOU-HAN-CYA0630-15UH_C5189959.html" (at 242.57 43.18 0)
+      (effects (font (size 1.27 1.27)) hide)
+    )
